Commit message: Adding new chassi and Nav2 navigation

File: urdf/robot.urdf (robot description, URDF)
Before this commit: robot robot, 6 links, 5 joints
Links:
- removed link caster_wheel
- added link caster_wheel_b_left, mass 0.1; collision sphere radius=0.035; visual sphere radius=0.035
- added link caster_wheel_b_right, mass 0.1; collision sphere radius=0.035; visual sphere radius=0.035
- added link caster_wheel_f_left, mass 0.1; collision sphere radius=0.035; visual sphere radius=0.035
- added link caster_wheel_f_right, mass 0.1; collision sphere radius=0.035; visual sphere radius=0.035
- link base_link: mass 1.0 -> 1.00000000; geometry collision mesh filename=file://$(find iris_description)/meshes/chassi_1.stl scale=1 1 1; visual mesh filename=file://$(find iris_description)/meshes/chassi_1.stl scale=1 1 1
- link laser_scanner: geometry collision cylinder length=0.03 radius=0.025; visual cylinder length=0.03 radius=0.025
Joints:
- removed joint caster_wheel_joint
- added joint caster_wheel_b_left_joint: type fixed, parent base_link, child caster_wheel_b_left, origin xyz=0.18 0.13 -0.05 rpy=0 0 0
- added joint caster_wheel_b_right_joint: type fixed, parent base_link, child caster_wheel_b_right, origin xyz=0.18 -0.13 -0.05 rpy=0 0 0
- added joint caster_wheel_f_left_joint: type fixed, parent base_link, child caster_wheel_f_left, origin xyz=-0.18 0.13 -0.05 rpy=0 0 0
- added joint caster_wheel_f_right_joint: type fixed, parent base_link, child caster_wheel_f_right, origin xyz=-0.18 -0.13 -0.05 rpy=0 0 0
- joint laser_scanner_joint: axis 0.0 1 0.0 -> 0.0 1 0; origin xyz=0.0 0.0 0.08 rpy=0.0 0.0 3.1415 -> xyz=0.21 0.0 0.005 rpy=0.0 0.0 0
- joint left_wheel_joint: axis 0.0 0.0 1 -> 0 0.0 -1; origin xyz=-0.2825 0.125 -0.05 rpy=1.5708 0.0 0.0 -> xyz=0 0.25 -0.05 rpy=1.5708 0.0 0.0
- joint right_wheel_joint: axis 0.0 0.0 1 -> 0 0.0 1; origin xyz=-0.2825 -0.125 -0.05 rpy=1.5708 0.0 0.0 -> xyz=0 -0.25 -0.05 rpy=-1.5708 0.0 0.0
